File: ZX Max 128 PlusD Issue1.kicad_pcb (KiCad board)
At the start: 2 copper layers, 213 x 130 mm, 272 parts, among them J1 8 Pin FFC Connector, J10 Header 2x1, J11 FDC Connector, J12 Header 2x2, J13 Header 2x2, J14 Header 4 Pin FDD Power, J15 PlusD ROM, J17 Header 2x1, J2 5 Pin FFC Connector, J3 ZX_48K_EDGE, J4 PJ-002A, J5 AV Jack, J6 Connector Audio 3525N, J7 A-DS_09_A_KG-T4S, J8 Connector 9 Pin Mini DIN, J9 Header 5x2, M1 MountingHole, M2 MountingHole, M3 MountingHole, M4 MountingHole, M5 MountingHole, M6 MountingHole, Q1 Transistor BC548, U1 Z80, U10 CD74HC30E, U11 74HC74, U12 CD74HC366E, U13 AD724JRZ, U14 R-78E5.0-1.0, U15 ESP8266-12E, U16 WD1772, U17 AS6C6264-55PCN, U18 EEPROM/EPROM 32Kx8, U19 GAL20V8B, U2 EEPROM/EPROM 32Kx8, U20 CD74HC30E, U21 74HC32, U22 Sound Generator SAA1099, U23 MCP602-I/P, U24 SAM2695, U25 3V3 1Amp, U26 74HC27, U27 74HC00, U28 SN74LS175NE4, U29 SN74LS06, U3 AS6C1008-55PCN, U30 74HC126, U4 AS6C1008-55PCN, U5 EPM7128SLC, U6 74HC04, U7 SN74HC174N, U8 AY-3-8910, U9 AY-3-8910, Y1 28.375Mhz, Y2 4.433Mhz, Y3 ECS-2100A-080, Y4 12Mhz, Y4x1 12Mhz, Y5 Crystal 8Mhz

Commit message: Add files via upload
Upload of Kicad 10 files, replacing those from Kicad 9.
Routing:
- net GND: track 1386.4 -> 1484.2 mm
- net VCC: track 934.1 -> 1002.2 mm
- net Luma: track 0.00 -> 12.0 mm
- net CLK28: vias 1 -> 0
